Commit message: Some update for the files

File: delta_robot_description/urdf/delta.xacro (robot description, xacro)
@@ -2,145 +2,118 @@
 <!-- Robot Name -->
 <robot name="delta_robot" xmlns:xacro="http://www.ros.org/wiki/xacro">
+  <!-- BGN - Include -->
+  <xacro:include filename="$(find delta_robot_description)/urdf/parameter_delta.xacro" />
+  <xacro:include filename="$(find delta_robot_description)/urdf/linkjoint_delta.xacro" />
+  <!-- END - Include -->
+<!-- Used for fixing robot to Gazebo 'base_link' -->
+  <link name="world">
+  </link>
+  <joint name="fixed" type="fixed">
+    <origin rpy="0 0 0" xyz="0 0 0" />
+    <parent link="world"/>
+    <child link="base_link"/>
+  </joint>
 <!-- Base -->
-    <link name="base_link">
-        <visual>
-            <geometry>
-                <cylinder length="0.02" radius="0.180"/>
-            </geometry>
-            <origin rpy="0 0 0" xyz="0 0 0"/>
-        </visual>
-    </link>
+ <m_link_cylinder name="${link_00_name}"
+              origin_rpy="0 0 0" origin_xyz="0 0 0"
+              mass="47"
+              ixx="1.765" ixy="0" ixz="0"
+              iyy="1.765" iyz="0"
+              izz="3.217"
+              radius="0.18" length="0.02" />
 <!-- Arm 1 -->
-    <link name="arm_1">
-        <visual>
-            <geometry>
-                <box size="0.300 0.02 0.02"/>
-            </geometry>
-            <origin rpy="0 0 0" xyz="0.150 0 0"/>
-            <material name="blue">
-                <color rgba="0 0 1 1"/>
-             </material>
-         </visual>
-    </link>
-    <joint name="base_to_arm_1" type="revolute">
-        <axis xyz="0 1 0"/>
-        <limit effort="1000.0" lower="-1.5708" upper="1.5708" velocity="0.5"/>
-        <parent link="base_link"/>
-        <child link="arm_1"/>
-        <origin rpy="0 0 -1.5708" xyz="0 -0.180 0"/>
-    </joint>
+ <m_joint name="joint1" type="revolute"
+           axis_xyz="0 1 0"
+           origin_rpy="0 0 -1.5708" origin_xyz="0 -0.180 0"
+           parent="base_link" child="arm_1"
+           limit_e="1000" limit_l="-1.5708" limit_u="1.5708" limit_v="0.5" />
+ <m_link_box name="${link_01_name}"
+              origin_rpy="0 0 0" origin_xyz="0.15 0 0"
+              mass="0.5"
+              ixx="0.065" ixy="0" ixz="0"
+              iyy="0.065" iyz="0"
+              izz="0.005"
+              size="0.3 0.02 0.02" />
  <!-- Down Part Arm 1 -->
-    <link name="down_arm_1">
-        <visual>
-            <geometry>
-                <box size="0.800 0.02 0.02"/>
-            </geometry>
-            <origin rpy="0 0 0" xyz="0.400 0 0"/>
-            <material name="blue">
-                <color rgba="0 0 0.8 1"/>
-            </material>
-        </visual>
-    </link>
-    <joint name="down_arm_1_to_arm_1" type="revolute">
-        <axis xyz="0 1 0"/>
-        <limit effort="1000.0" lower="-1.5708" upper="1.5708" velocity="0.5"/>
-        <parent link="arm_1"/>
-        <child link="down_arm_1"/>
-        <origin rpy="0 1.5708 0" xyz="0.300 0 0"/>
-    </joint>
+   <m_joint name="joint2" type="revolute"
+           axis_xyz="0 1 0"
+           origin_rpy="0 1.5708 0" origin_xyz="0.300 0 0"
+           parent="arm_1" child="down_arm_1"
+           limit_e="1000" limit_l="-1.5708" limit_u="1.5708" limit_v="0.5" />
+  <m_link_box name="${link_02_name}"
+              origin_rpy="0 0 0" origin_xyz="0.4 0 0"
+              mass="0.5"
+              ixx="0.065" ixy="0" ixz="0"
+              iyy="0.065" iyz="0"
+              izz="0.005"
+              size="0.8 0.02 0.02" />
     <!-- End efector -->
-    <link name="tool0">
-        <visual>
-            <geometry>
-                <cylinder length="0.02" radius="0.100"/>
-            </geometry>
-            <origin rpy="0 0 0" xyz="0.100 0 0"/>
-             <material name="green">
-                <color rgba="0 0.8 0 1"/>
-            </material>
-        </visual>
-    </link>
-    <joint name="tool0_to_down_arm_1" type="revolute">
-        <axis xyz="0 1 0"/>
-        <limit effort="1000.0" lower="-1.5708" upper="1.5708" velocity="0.5"/>
-        <parent link="down_arm_1"/>
-        <child link="tool0"/>
-        <origin rpy="0 1.5708 0" xyz="0.800 0 0"/>
-     </joint>
+  <m_joint name="joint3" type="revolute"
+           axis_xyz="0 1 0"
+           origin_rpy="0 1.5708 0" origin_xyz="0.800 0 0"
+           parent="down_arm_1" child="tool0"
+           limit_e="1000" limit_l="-1.5708" limit_u="1.5708" limit_v="0.5" />
+ <m_link_tool name="${link_03_name}"
+              origin_rpy="0 0 0" origin_xyz="0.1 0 0"
+              mass="47"
+              ixx="1.765" ixy="0" ixz="0"
+              iyy="1.765" iyz="0"
+              izz="3.217"
+              radius="0.100" length="0.02" />
     <!-- Arm 2 -->
-    <link name="arm_2">
-        <visual>
-         <geometry>
-            <box size="0.300 0.02 0.02"/>
-        </geometry>
-        <origin rpy="0 0 0" xyz="0.150 0 0"/>
-        <material name="blue">
-            <color rgba="0 0 1 1"/>
-        </material>
-        </visual>
-    </link>
-    <joint name="base_to_arm_2" type="revolute">
-        <axis xyz="0 1 0"/>
-        <limit effort="1000.0" lower="-1.5708" upper="1.5708" velocity="0.5"/>
-        <parent link="base_link"/>
-        <child link="arm_2"/>
-        <origin rpy="0 0 0.5236" xyz="0.155885 0.09 0"/>
-    </joint>
+ <m_joint name="joint4" type="revolute"
+           axis_xyz="0 1 0"
+           origin_rpy="0 0 0.5236" origin_xyz="0.155885 0.09 0"
+           parent="base_link" child="arm_2"
+           limit_e="1000" limit_l="-1.5708" limit_u="1.5708" limit_v="0.5" />
+ <m_link_box name="${link_04_name}"
+              origin_rpy="0 0 0" origin_xyz="0.15 0 0"
+              mass="0.5"
+              ixx="0.065" ixy="0" ixz="0"
+              iyy="0.065" iyz="0"
+              izz="0.005"
+              size="0.3 0.02 0.02" />
 <!-- Down Part Arm 2 -->
-    <link name="down_arm_2">
-         <visual>
-            <geometry>
-                <box size="0.800 0.02 0.02"/>
-            </geometry>
-            <origin rpy="0 0 0" xyz="0.400 0 0"/>
-            <material name="blue">
-                <color rgba="0 0 0.8 1"/>
-             </material>
-        </visual>
-    </link>
-    <joint name="down_arm_2_to_arm_2" type="revolute">
-        <axis xyz="0 1 0"/>
-        <limit effort="1000.0" lower="-1.5708" upper="1.5708" velocity="0.5"/>
-        <parent link="arm_2"/>
-        <child link="down_arm_2"/>
-        <origin rpy="0 1.5708 0" xyz="0.300 0 0"/>
-    </joint>
+   <m_joint name="joint5" type="revolute"
+           axis_xyz="0 1 0"
+           origin_rpy="0 1.5708 0" origin_xyz="0.300 0 0"
+           parent="arm_2" child="down_arm_2"
+           limit_e="1000" limit_l="-1.5708" limit_u="1.5708" limit_v="0.5" />
+  <m_link_box name="${link_05_name}"
+              origin_rpy="0 0 0" origin_xyz="0.4 0 0"
+              mass="0.5"
+              ixx="0.065" ixy="0" ixz="0"
+              iyy="0.065" iyz="0"
+              izz="0.005"
+              size="0.8 0.02 0.02" />
     <!-- Arm 3 -->
-    <link name="arm_3">
-        <visual>
-            <geometry>
-                <box size="0.300 0.02 0.02"/>
-            </geometry>
-            <origin rpy="0 0 0" xyz="0.150 0 0"/>
-            <material name="blue">
-                <color rgba="0 0 1 1"/>
-            </material>
-        </visual>
-    </link>
-    <joint name="base_to_arm_3" type="revolute">
-        <axis xyz="0 1 0"/>
-        <limit effort="1000.0" lower="-1.5708" upper="1.5708" velocity="0.5"/>
-        <parent link="base_link"/>
-        <child link="arm_3"/>
-        <origin rpy="0 0 2.618" xyz="-0.155885 0.09 0"/>
-    </joint>
+<m_joint name="joint6" type="revolute"
+           axis_xyz="0 1 0"
+           origin_rpy="0 0 2.618" origin_xyz="-0.155885 0.09 0"
+           parent="base_link" child="arm_3"
+           limit_e="1000" limit_l="-1.5708" limit_u="1.5708" limit_v="0.5" />
+ <m_link_box name="${link_06_name}"
+              origin_rpy="0 0 0" origin_xyz="0.15 0 0"
+              mass="0.5"
+              ixx="0.065" ixy="0" ixz="0"
+              iyy="0.065" iyz="0"
+              izz="0.005"
+              size="0.3 0.02 0.02" />
 <!-- Down Part Arm 3 -->
-    <link name="down_arm_3">
-        <visual>
-            <geometry>
-                <box size="0.800 0.02 0.02"/>
-            </geometry>
-            <origin rpy="0 0 0" xyz="0.400 0 0"/>
-            <material name="blue">
-                <color rgba="0 0 0.8 1"/>
-            </material>
-        </visual>
-    </link>
-    <joint name="down_arm_3_to_arm_3" type="revolute">
-        <axis xyz="0 1 0"/>
-        <limit effort="1000.0" lower="-1.5708" upper="1.5708" velocity="0.5"/>
-        <parent link="arm_3"/>
-        <child link="down_arm_3"/>
-        <origin rpy="0 1.5708 0" xyz="0.300 0 0"/>
-    </joint>
+   <m_joint name="joint7" type="revolute"
+           axis_xyz="0 1 0"
+           origin_rpy="0 1.5708 0" origin_xyz="0.300 0 0"
+           parent="arm_3" child="down_arm_3"
+           limit_e="1000" limit_l="-1.5708" limit_u="1.5708" limit_v="0.5" />
+  <m_link_box name="${link_07_name}"
+              origin_rpy="0 0 0" origin_xyz="0.4 0 0"
+              mass="0.5"
+              ixx="0.065" ixy="0" ixz="0"
+              iyy="0.065" iyz="0"
+              izz="0.005"
+              size="0.8 0.02 0.02" />
+    <gazebo>
+    <plugin name="gazebo_ros_control" filename="libgazebo_ros_control.so">
+    </plugin>
+    </gazebo>
 </robot>
